File: keypad-prototype/keypad-base/keypad-base.kicad_pcb (KiCad board)
At the start: 2 copper layers, 150.2 x 64.2 mm, 66 parts, among them CON1 AVR-ISP-6, J1 USB_C_Receptacle_USB2.0, J2 Conn_01x02, J3 Conn_01x02, Q1 AO3400A, SW1 Switch_SW_Push, SW2 Switch_SW_Push, SW3 Switch_SW_Push, SW4 Switch_SW_Push, SW5 Switch_SW_Push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

Commit message: keypad-base/keypad-frame: change to M2 standoffs, Apr2021a release
Parts:
- H2, H3, H4, H5: footprint tom-mechanical:STUD_SOLDER_M3 -> tom-mechanical:STUD_SOLDER_M2_WURTH

Commit message: keypad-base: Jun2021 - change standoff type
Parts:
- H2, H3, H4, H5: footprint tom-mechanical:STUD_SOLDER_M2_WURTH -> tom-mechanical:STUD_SOLDER_SMTSO_M3
Routing:
- net +5V: track 269.1 -> 280.0 mm
Changed lines of the file:
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@@
     (thickness 1.6)
     (drawings 22)
-    (tracks 881)
+    (tracks 883)
     (zones 0)
     (modules 66)
@@
   (page A4)
   (title_block
-    (date 2021-04-25)
-    (rev Apr2021a)
+    (date 2021-06-05)
+    (rev Jun2021)
   )
   (layers
     (0 F.Cu signal)
-    (31 B.Cu signal hide)
+    (31 B.Cu signal)
     (32 B.Adhes user hide)
     (33 F.Adhes user)
     (34 B.Paste user hide)
     (35 F.Paste user)
-    (36 B.SilkS user hide)
+    (36 B.SilkS user)
     (37 F.SilkS user)
     (38 B.Mask user hide)
@@
   )
   (setup
-    (last_trace_width 0.25)
+    (last_trace_width 1)
     (user_trace_width 0.5)
     (user_trace_width 1)
@@
     (add_net "Net-(U8-Pad2)")
   )
-  (module tom-mechanical:STUD_SOLDER_M2_WURTH (layer B.Cu)
+  (module tom-mechanical:STUD_SOLDER_SMTSO_M3 (layer B.Cu)
     (at 107.5 111.9)
-    (descr "SMD Standoff Wurth 9774040243R M2")
+    (descr "SMD Standoff Aliexpress")
     (attr smd)
     (fp_text reference H5 (at 0 -0.5) (layer B.SilkS) hide
@@
       (effects (font (size 1 1) (thickness 0.15)) (justify mirror))
     )
-    (pad 1 thru_hole circle (at 0 0) (size 3.2 3.2) (drill 3.2) (layers *.Cu *.Mask))
-    (pad 1 smd circle (at 0 0) (size 6 6) (layers B.Cu B.Paste B.Mask))
+    (pad 1 thru_hole circle (at 0 0) (size 7 7) (drill 4.2) (layers *.Cu *.Mask))
+    (model /home/tom/git/TomKeddie/prj-pcb-experiments/tom-kicad/footprints/3dmodels/SMTSO-M3-10ET-PennEngineering-3D-05-29-2021.stp
+      (offset (xyz 0 0 -1.6))
+      (scale (xyz 1 1 1))
+      (rotate (xyz 0 90 0))
+    )
   )
-  (module tom-mechanical:STUD_SOLDER_M2_WURTH (layer B.Cu)
+  (module tom-mechanical:STUD_SOLDER_SMTSO_M3 (layer B.Cu)
     (at 107.5 59.9)
-    (descr "SMD Standoff Wurth 9774040243R M2")
+    (descr "SMD Standoff Aliexpress")
     (attr smd)
     (fp_text reference H4 (at 0 -0.5) (layer B.SilkS) hide
@@
       (effects (font (size 1 1) (thickness 0.15)) (justify mirror))
     )
-    (pad 1 thru_hole circle (at 0 0) (size 3.2 3.2) (drill 3.2) (layers *.Cu *.Mask))
-    (pad 1 smd circle (at 0 0) (size 6 6) (layers B.Cu B.Paste B.Mask))
+    (pad 1 thru_hole circle (at 0 0) (size 7 7) (drill 4.2) (layers *.Cu *.Mask))
+    (model /home/tom/git/TomKeddie/prj-pcb-experiments/tom-kicad/footprints/3dmodels/SMTSO-M3-10ET-PennEngineering-3D-05-29-2021.stp
+      (offset (xyz 0 0 -1.6))
+      (scale (xyz 1 1 1))
+      (rotate (xyz 0 90 0))
+    )
   )
-  (module tom-mechanical:STUD_SOLDER_M2_WURTH (layer B.Cu)
+  (module tom-mechanical:STUD_SOLDER_SMTSO_M3 (layer B.Cu)
     (at 225.5 59.9)
-    (descr "SMD Standoff Wurth 9774040243R M2")
+    (descr "SMD Standoff Aliexpress")
     (attr smd)
     (fp_text reference H3 (at 0 -0.5) (layer B.SilkS) hide
@@
       (effects (font (size 1 1) (thickness 0.15)) (justify mirror))
     )
-    (pad 1 thru_hole circle (at 0 0) (size 3.2 3.2) (drill 3.2) (layers *.Cu *.Mask))
-    (pad 1 smd circle (at 0 0) (size 6 6) (layers B.Cu B.Paste B.Mask))
+    (pad 1 thru_hole circle (at 0 0) (size 7 7) (drill 4.2) (layers *.Cu *.Mask))
+    (model /home/tom/git/TomKeddie/prj-pcb-experiments/tom-kicad/footprints/3dmodels/SMTSO-M3-10ET-PennEngineering-3D-05-29-2021.stp
+      (offset (xyz 0 0 -1.6))
+      (scale (xyz 1 1 1))
+      (rotate (xyz 0 90 0))
+    )
   )
-  (module tom-mechanical:STUD_SOLDER_M2_WURTH (layer B.Cu)
+  (module tom-mechanical:STUD_SOLDER_SMTSO_M3 (layer B.Cu)
     (at 225.5 111.9)
-    (descr "SMD Standoff Wurth 9774040243R M2")
+    (descr "SMD Standoff Aliexpress")
     (attr smd)
     (fp_text reference H2 (at 0 -0.5) (layer B.SilkS) hide
@@
       (effects (font (size 1 1) (thickness 0.15)) (justify mirror))
     )
-    (pad 1 thru_hole circle (at 0 0) (size 3.2 3.2) (drill 3.2) (layers *.Cu *.Mask))
-    (pad 1 smd circle (at 0 0) (size 6 6) (layers B.Cu B.Paste B.Mask))
+    (pad 1 thru_hole circle (at 0 0) (size 7 7) (drill 4.2) (layers *.Cu *.Mask))
+    (model /home/tom/git/TomKeddie/prj-pcb-experiments/tom-kicad/footprints/3dmodels/SMTSO-M3-10ET-PennEngineering-3D-05-29-2021.stp
+      (offset (xyz 0 0 -1.6))
+      (scale (xyz 1 1 1))
+      (rotate (xyz 0 90 0))
+    )
   )
   (module tom-passives:R_0805_2012Metric (layer F.Cu)
@@
   (segment (start 166.37 61.214) (end 162.13293 61.214) (width 1) (layer F.Cu) (net 24))
   (segment (start 162.13293 61.214) (end 161.466907 61.880023) (width 1) (layer F.Cu) (net 24))
-  (segment (start 108.712 63.5) (end 110.998 61.214) (width 1) (layer F.Cu) (net 24))
-  (segment (start 110.998 61.214) (end 115.316 61.214) (width 1) (layer F.Cu) (net 24))
-  (segment (start 103.632 63.5) (end 108.712 63.5) (width 1) (layer F.Cu) (net 24))
-  (segment (start 94.996 72.136) (end 103.632 63.5) (width 1) (layer F.Cu) (net 24))
-  (segment (start 94.996 81.026) (end 94.996 72.136) (width 1) (layer F.Cu) (net 24))
+  (segment (start 113.284 55.372) (end 115.316 57.404) (width 1) (layer F.Cu) (net 24))
+  (segment (start 105.156 55.372) (end 113.284 55.372) (width 1) (layer F.Cu) (net 24))
+  (segment (start 103.124 57.404) (end 105.156 55.372) (width 1) (layer F.Cu) (net 24))
+  (segment (start 103.124 61.976) (end 103.124 57.404) (width 1) (layer F.Cu) (net 24))
+  (segment (start 94.996 70.104) (end 103.124 61.976) (width 1) (layer F.Cu) (net 24))
+  (segment (start 115.316 57.404) (end 115.316 61.214) (width 1) (layer F.Cu) (net 24))
+  (segment (start 94.996 81.026) (end 94.996 70.104) (width 1) (layer F.Cu) (net 24))
   (segment (start 164.5 84.971022) (end 164.5 84.4855) (width 0.25) (layer F.Cu) (net 25))
   (segment (start 164.136032 85.33499) (end 164.5 84.971022) (width 0.25) (layer F.Cu) (net 25))
